Commit message: fix in simulations

File: franka_simulation/urdf/obstacles/multi_obstacle_scene.urdf.xacro (robot description, xacro)
@@ -31,4 +31,5 @@
     </visual>
     <collision>
+      <origin xyz="0 0 0" rpy="0 0 0"/>
       <geometry>
         <box size="$(arg box1_size_x) $(arg box1_size_y) $(arg box1_size_z)"/>
@@ -48,4 +49,9 @@
     <material>Gazebo/Red</material>
     <static>true</static>
+    <!-- Contact parameters (Gazebo-classic style; kept for parity even if ignored by gz-sim) -->
+    <mu1>1.0</mu1>
+    <mu2>1.0</mu2>
+    <kp>1e7</kp>
+    <kd>1.0</kd>
   </gazebo>
   <!-- ========================================== -->
@@ -60,4 +66,5 @@
   <link name="obstacle_box_lateral" >
     <visual>
+      <origin xyz="0 0 0" rpy="0 0 0"/>
       <geometry>
         <box size="$(arg box2_size_x) $(arg box2_size_y) $(arg box2_size_z)"/>
@@ -68,4 +75,5 @@
     </visual>
     <collision>
+      <origin xyz="0 0 0" rpy="0 0 0"/>
       <geometry>
         <box size="$(arg box2_size_x) $(arg box2_size_y) $(arg box2_size_z)"/>
@@ -85,4 +93,9 @@
     <material>Gazebo/Yellow</material>
     <static>true</static>
+    <!-- Match central obstacle contact params -->
+    <mu1>1.0</mu1>
+    <mu2>1.0</mu2>
+    <kp>1e7</kp>
+    <kd>1.0</kd>
   </gazebo>
   <!-- ========================================== -->
